File: bottom_board_palmtop/usb.kicad_sch (KiCad schematic)
At the start: 40 parts, among them J1 Left USB, J2 Right USB, J3 Center USB, SW3 SW_EN, U1 TPAZ1043-04F, U26 TPAZ1043-04F, U27 WUSB3801Q-12/TR, U29 WUSB3801Q-12/TR, U3 TPAZ1043-04F, U30 SY6280AAAC, U31 SY6280AAAC, U32 PI3USB42ZMEX, U33 FUSB302B01MPX, U35 PI3USB42ZMEX

Commit message: bottom_board_palmtop: JLC PCBA preparation; clarifying I2C addresses in use
Parts:
- Green1, Green2: value LED 0603 -> LED 0603 Green; LCSC Part C965801 -> (none)
- J1, J2: LCSC Part (none) -> C3039315
- J3: LCSC Part (none) -> C165948
Changed lines of the file:
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@@
 			)
 		)
+		(property "LCSC Part" "C3039315"
+			(at 24.13 124.46 0)
+			(effects
+				(font
+					(size 1.27 1.27)
+				)
+				(hide yes)
+			)
+		)
 		(pin "A5"
 		)
@@
 			)
 		)
+		(property "LCSC Part" "C165948"
+			(at 143.51 29.21 90)
+			(effects
+				(font
+					(size 1.27 1.27)
+				)
+				(hide yes)
+			)
+		)
 		(pin "B9"
 		)
@@
 			)
 		)
+		(property "LCSC Part" "C3039315"
+			(at 265.43 118.11 0)
+			(effects
+				(font
+					(size 1.27 1.27)
+				)
+				(hide yes)
+			)
+		)
 		(pin "A5"
 		)
@@
 			)
 		)
-		(property "Value" "LED 0603"
+		(property "Value" "LED 0603 Green"
 			(at 95.25 171.196 0)
 			(effects
@@
 			)
 		)
-		(property "LCSC Part" "C965801"
+		(property "LCSC Part" ""
 			(at 92.71 171.45 0)
 			(effects
@@
 			)
 		)
-		(property "Value" "LED 0603"
+		(property "Value" "LED 0603 Green"
 			(at 182.88 140.716 0)
 			(effects
@@
 			)
 		)
-		(property "LCSC Part" "C965801"
+		(property "LCSC Part" ""
 			(at 185.42 140.97 0)
 			(effects
